File: ESPWatchS3.kicad_pcb (KiCad board)
At the start: 4 copper layers, 0 parts

Commit message: Fixed footprints, dumped parts into PCB layout
Parts:
- added ANT1: W3008G, WatchParts:ANTENNA_W3008, F.Cu at (122.5, 45.7)
- added ANT2: 1575AT43A0040E, WatchParts:1575AT43A0040E, F.Cu at (107.5, 108.0)
- added BT1: RJD3048, WatchParts:BAT_3046, F.Cu at (98.1, 57.7)
- added C1: 0.1u, Capacitor_SMD:C_0402_1005Metric, F.Cu at (104.5, 83.0)
- added C10: 0.1u, Capacitor_SMD:C_0402_1005Metric, F.Cu at (107.3, 85.0)
- added C11: 0.1u, Capacitor_SMD:C_0402_1005Metric, F.Cu at (107.3, 87.0)
- added C12: 0.1u, Capacitor_SMD:C_0402_1005Metric, F.Cu at (107.3, 88.9)
- added C13: 0.1u, Capacitor_SMD:C_0402_1005Metric, F.Cu at (107.3, 90.9)
- added C14: 0.1u, Capacitor_SMD:C_0402_1005Metric, F.Cu at (107.3, 92.9)
- added C15: 0.1u, Capacitor_SMD:C_0402_1005Metric, F.Cu at (107.3, 94.8)
- added C16: 0.1u, Capacitor_SMD:C_0402_1005Metric, F.Cu at (107.3, 96.8)
- added C17: 1u, Capacitor_SMD:C_0603_1608Metric, F.Cu at (87.6, 88.8)
- added C18: 1u, Capacitor_SMD:C_0603_1608Metric, F.Cu at (87.6, 91.3)
- added C19: 1u, Capacitor_SMD:C_0603_1608Metric, F.Cu at (87.6, 93.8)
- added C2: 0.1u, Capacitor_SMD:C_0402_1005Metric, F.Cu at (104.5, 85.0)
- added C20: 1u, Capacitor_SMD:C_0603_1608Metric, F.Cu at (87.6, 96.3)
- added C21: 1u, Capacitor_SMD:C_0603_1608Metric, F.Cu at (87.6, 98.8)
- added C22: 1u, Capacitor_SMD:C_0603_1608Metric, F.Cu at (87.6, 101.4)
- added C23: 1u, Capacitor_SMD:C_0603_1608Metric, F.Cu at (91.6, 88.8)
- added C24: 1u, Capacitor_SMD:C_0603_1608Metric, F.Cu at (91.6, 91.3)
- added C25: 1u, Capacitor_SMD:C_0603_1608Metric, F.Cu at (91.6, 93.8)
- added C26: 1u, Capacitor_SMD:C_0603_1608Metric, F.Cu at (91.6, 96.3)
- added C27: 1u, Capacitor_SMD:C_0603_1608Metric, F.Cu at (91.6, 98.8)
- added C28: 10u, Capacitor_SMD:C_0805_2012Metric, F.Cu at (116.8, 83.5)
- added C29: 10u, Capacitor_SMD:C_0805_2012Metric, F.Cu at (116.8, 86.6)
- added C3: 0.1u, Capacitor_SMD:C_0402_1005Metric, F.Cu at (104.5, 87.0)
- added C30: 10u, Capacitor_SMD:C_0805_2012Metric, F.Cu at (116.8, 89.6)
- added C31: 10u, Capacitor_SMD:C_0805_2012Metric, F.Cu at (116.8, 92.6)
- added C32: 10u, Capacitor_SMD:C_0805_2012Metric, F.Cu at (116.8, 95.6)
- added C33: 10u, Capacitor_SMD:C_0805_2012Metric, F.Cu at (121.2, 83.5)
- added C34: 10u, Capacitor_SMD:C_0805_2012Metric, F.Cu at (121.2, 86.6)
- added C35: 10u, Capacitor_SMD:C_0805_2012Metric, F.Cu at (121.2, 89.6)
- added C36: 0.01u, Capacitor_SMD:C_0402_1005Metric, F.Cu at (110.2, 83.0)
- added C37: 0.01u, Capacitor_SMD:C_0402_1005Metric, F.Cu at (110.2, 85.0)
- added C38: 0.01u, Capacitor_SMD:C_0402_1005Metric, F.Cu at (110.2, 87.0)
- added C39: 0.01u, Capacitor_SMD:C_0402_1005Metric, F.Cu at (110.2, 88.9)
- added C4: 0.1u, Capacitor_SMD:C_0402_1005Metric, F.Cu at (104.5, 88.9)
- added C40: 0.01u, Capacitor_SMD:C_0402_1005Metric, F.Cu at (110.2, 90.9)
- added C41: 0.01u, Capacitor_SMD:C_0402_1005Metric, F.Cu at (110.2, 92.9)
- added C42: 0.01u, Capacitor_SMD:C_0402_1005Metric, F.Cu at (110.2, 94.8)
- added C43: 3.9p, Capacitor_SMD:C_0402_1005Metric, F.Cu at (110.2, 96.8)
- added C44: 4.8p, Capacitor_SMD:C_0402_1005Metric, F.Cu at (113.1, 83.0)
- added C45: 18p, Capacitor_SMD:C_0402_1005Metric, F.Cu at (113.1, 85.0)
- added C46: 18p, Capacitor_SMD:C_0402_1005Metric, F.Cu at (113.1, 87.0)
- added C47: 10p, Capacitor_SMD:C_0402_1005Metric, F.Cu at (113.1, 88.9)
- added C48: 10p, Capacitor_SMD:C_0402_1005Metric, F.Cu at (113.1, 90.9)
- added C49: 22u, Capacitor_SMD:C_0805_2012Metric, F.Cu at (121.2, 92.6)
- added C5: 0.1u, Capacitor_SMD:C_0402_1005Metric, F.Cu at (104.5, 90.9)
- added C50: 47u, Capacitor_SMD:C_0805_2012Metric, F.Cu at (121.2, 95.6)
- added C51: DNF, Capacitor_SMD:C_0402_1005Metric, F.Cu at (113.1, 92.9)
- added C52: 2p, Capacitor_SMD:C_0402_1005Metric, F.Cu at (113.1, 94.8)
- added C53: 0.001u, Capacitor_SMD:C_0402_1005Metric, F.Cu at (113.1, 96.8)
- added C6: 0.1u, Capacitor_SMD:C_0402_1005Metric, F.Cu at (104.5, 92.9)
- added C7: 0.1u, Capacitor_SMD:C_0402_1005Metric, F.Cu at (104.5, 94.8)
- added C8: 0.1u, Capacitor_SMD:C_0402_1005Metric, F.Cu at (104.5, 96.8)
- added C9: 0.1u, Capacitor_SMD:C_0402_1005Metric, F.Cu at (107.3, 83.0)
- added D1: MBR0530, Diode_SMD:D_SOD-123, F.Cu at (117.4, 108.8)
- added D2: Status 1, LED_SMD:LED_0603_1608Metric, F.Cu at (127.1, 59.1)
- added D3: Status 2, LED_SMD:LED_0603_1608Metric, F.Cu at (127.1, 61.6)
- added FL1: B39162B4327P810, WatchParts:FIL_B39162B4327P810, F.Cu at (128.1, 102.0)
- added J1: USB, Connector_USB:USB_C_Receptacle_GCT_USB4105-xx-A_16P_TopMnt_Horizontal, F.Cu at (120.4, 102.4)
- added J2: OLED, WatchParts:CS050Z24GA0, F.Cu at (113.1, 78.0)
- added J3: UART0, Connector_PinHeader_2.54mm:PinHeader_1x05_P2.54mm_Vertical, F.Cu at (125.8, 84.4)
- added JP1: VDD_3V3, Jumper:SolderJumper-2_P1.3mm_Open_RoundedPad1.0x1.5mm, F.Cu at (127.8, 43.6)
- added L1: 1.8n, Inductor_SMD:L_0402_1005Metric, F.Cu at (87.0, 74.6)
- added L2: DNF, Inductor_SMD:L_0402_1005Metric, F.Cu at (87.0, 76.6)
- added L3: 9.1n, Inductor_SMD:L_0402_1005Metric, F.Cu at (87.0, 78.6)
- added L4: 2.2n, Inductor_SMD:L_0402_1005Metric, F.Cu at (87.0, 80.6)
- added L5: 10u, Inductor_SMD:L_1008_2520Metric, F.Cu at (122.8, 109.0)
- added L6: 1u, WatchParts:SRP2512TMA1R0M, F.Cu at (122.7, 50.4)
- added Q1: DMN2050LFDB, WatchParts:MOSFET_DMP2160UFDB-7, F.Cu at (122.2, 70.8)
- added R1: 5.1k, Resistor_SMD:R_0402_1005Metric, F.Cu at (87.0, 82.6)
- added R10: 100k, Resistor_SMD:R_0402_1005Metric, F.Cu at (90.0, 86.6)
- added R11: 100k, Resistor_SMD:R_0402_1005Metric, F.Cu at (92.9, 74.6)
- added R12: 100k, Resistor_SMD:R_0402_1005Metric, F.Cu at (92.9, 76.6)
- added R13: 100k, Resistor_SMD:R_0402_1005Metric, F.Cu at (92.9, 78.6)
- added R14: 100k, Resistor_SMD:R_0402_1005Metric, F.Cu at (92.9, 80.6)
- added R15: 100k, Resistor_SMD:R_0402_1005Metric, F.Cu at (92.9, 82.6)
- added R16: 100k, Resistor_SMD:R_0402_1005Metric, F.Cu at (92.9, 84.6)
- added R17: 2.2k, Resistor_SMD:R_0402_1005Metric, F.Cu at (92.9, 86.6)
- added R18: 2.2k, Resistor_SMD:R_0402_1005Metric, F.Cu at (95.8, 74.6)
- added R19: 10m, Resistor_SMD:R_0805_2012Metric, F.Cu at (122.0, 64.5)
- added R2: 5.1k, Resistor_SMD:R_0402_1005Metric, F.Cu at (87.0, 84.6)
- added R20: 10m, Resistor_SMD:R_0805_2012Metric, F.Cu at (122.0, 67.5)
- added R21: 10k, Resistor_SMD:R_0402_1005Metric, F.Cu at (95.8, 76.6)
- added R22: 10k, Resistor_SMD:R_0402_1005Metric, F.Cu at (95.8, 78.6)
- added R23: 10k, Resistor_SMD:R_0402_1005Metric, F.Cu at (95.8, 80.6)
- added R24: 100R, Resistor_SMD:R_0402_1005Metric, F.Cu at (95.8, 82.6)
- added R25: 22R, Resistor_SMD:R_0402_1005Metric, F.Cu at (95.8, 84.6)
- added R26: DNF, Resistor_SMD:R_0402_1005Metric, F.Cu at (95.8, 86.6)
- added R27: 20nH, Resistor_SMD:R_0402_1005Metric, F.Cu at (98.7, 74.6)
- added R28: 330R, Resistor_SMD:R_0402_1005Metric, F.Cu at (98.7, 76.6)
- added R29: 330R, Resistor_SMD:R_0402_1005Metric, F.Cu at (98.7, 78.6)
- added R3: 100k, Resistor_SMD:R_0402_1005Metric, F.Cu at (87.0, 86.6)
- added R30: 1k, Resistor_SMD:R_0402_1005Metric, F.Cu at (98.7, 80.6)
- added R31: 9.1k, Resistor_SMD:R_0402_1005Metric, F.Cu at (98.7, 82.6)
- added R32: 470R, Resistor_SMD:R_0402_1005Metric, F.Cu at (98.7, 84.6)
- added R33: 10k, Resistor_SMD:R_0402_1005Metric, F.Cu at (98.7, 86.6)
- added R34: 511k, Resistor_SMD:R_0402_1005Metric, F.Cu at (101.6, 74.6)
- added R35: 91k, Resistor_SMD:R_0402_1005Metric, F.Cu at (101.6, 76.6)
- added R36: DNF, Resistor_SMD:R_0402_1005Metric, F.Cu at (101.6, 78.6)
- added R37: 1.6k, Resistor_SMD:R_0402_1005Metric, F.Cu at (101.6, 80.6)
- added R38: 6.2k, Resistor_SMD:R_0402_1005Metric, F.Cu at (101.6, 82.6)
- added R39: 1M, Resistor_SMD:R_0402_1005Metric, F.Cu at (101.6, 84.6)
- added R4: 100k, Resistor_SMD:R_0402_1005Metric, F.Cu at (90.0, 74.6)
- added R5: 100k, Resistor_SMD:R_0402_1005Metric, F.Cu at (90.0, 76.6)
- added R6: 100k, Resistor_SMD:R_0402_1005Metric, F.Cu at (90.0, 78.6)
- added R7: 100k, Resistor_SMD:R_0402_1005Metric, F.Cu at (90.0, 80.6)
- added R8: 100k, Resistor_SMD:R_0402_1005Metric, F.Cu at (90.0, 82.6)
- added R9: 100k, Resistor_SMD:R_0402_1005Metric, F.Cu at (90.0, 84.6)
- added SW1: Reset, WatchParts:PTS815SJM250SMTRLFS, F.Cu at (81.3, 76.8)
- added SW2: Boot, WatchParts:PTS815SJM250SMTRLFS, F.Cu at (81.3, 83.1)
- added SW3: User 1, WatchParts:PTS815SJM250SMTRLFS, F.Cu at (81.3, 89.4)
- added SW4: User 2, WatchParts:PTS815SJM250SMTRLFS, F.Cu at (81.3, 95.7)
- added SW5: User 3, WatchParts:PTS815SJM250SMTRLFS, F.Cu at (81.3, 102.0)
- added SW6: User 4, WatchParts:PTS815SJM250SMTRLFS, F.Cu at (81.3, 108.3)
- added TP1: VOLED, TestPoint:TestPoint_Pad_D1.5mm, F.Cu at (95.4, 89.3)
- added TP2: VBATT, TestPoint:TestPoint_Pad_D1.5mm, F.Cu at (95.4, 92.9)
- added TP3: VMAIN, TestPoint:TestPoint_Pad_D1.5mm, F.Cu at (95.4, 96.4)
- added TP4: VSYS, TestPoint:TestPoint_Pad_D1.5mm, F.Cu at (95.4, 100.0)
- added TP5: GNSS_RESET, TestPoint:TestPoint_Pad_D1.5mm, F.Cu at (98.9, 89.3)
- added TP6: GNSS_SB, TestPoint:TestPoint_Pad_D1.5mm, F.Cu at (98.9, 92.9)
- added TP7: VUSB, TestPoint:TestPoint_Pad_D1.5mm, F.Cu at (98.9, 96.4)
- added U1: ESP32-S3R8, Package_DFN_QFN:QFN-56-1EP_7x7mm_P0.4mm_EP4x4mm, F.Cu at (98.2, 106.4)
- added U10: BD48KxxG, Package_TO_SOT_SMD:SOT-23, F.Cu at (126.6, 69.7)
- added U11: NJG1143UA2-TE1, WatchParts:AMP_NJG1143UA2-TE1, F.Cu at (128.0, 104.7)
- added U2: EVA-M8Q-0, WatchParts:LGA43R65P9X9_700X700X116, F.Cu at (107.6, 102.1)
- added U3: BME280, Package_LGA:Bosch_LGA-8_2.5x2.5mm_P0.65mm_ClockwisePinNumbering, F.Cu at (127.2, 109.2)
- added U4: TPS631000DRLR, WatchParts:SOTFL50P160X60-8N, F.Cu at (128.0, 98.9)
- added U5: AP3012, Package_TO_SOT_SMD:SOT-23-5, F.Cu at (126.7, 65.3)
- added U6: BQ298012, WatchParts:QFN50P150X150X40-8N, F.Cu at (128.2, 54.8)
- added U7: BQ27441-G1A, Package_SON:Texas_S-PDSO-N12, F.Cu at (122.9, 55.4)
- added U8: BQ24075RGTR, Package_DFN_QFN:VQFN-16-1EP_3x3mm_P0.5mm_EP1.8x1.8mm, F.Cu at (122.4, 60.4)
- added U9: IS25LP128F-JKLE, Package_SON:WSON-8-1EP_6x5mm_P1.27mm_EP3.4x4mm, F.Cu at (89.4, 105.9)
- added Y1: 40MHz, WatchParts:OSC_XRCGB40M000F1S1DR0, F.Cu at (127.8, 49.4)
- added Y2: 32.768kHz, Crystal:Crystal_SMD_3215-2Pin_3.2x1.5mm, F.Cu at (125.8, 75.3)
- added Y3: 32.768kHz, Crystal:Crystal_SMD_3215-2Pin_3.2x1.5mm, F.Cu at (125.8, 78.7)

Commit message: Initial PCB Stuff
Parts:
- moved BT1 74.4 mm to (140.0, 119.2), turned to 180 degrees
- moved FL1 47.6 mm to (84.4, 83.0)
- moved J1 47.6 mm to (76.7, 83.5)
- moved L5 47.6 mm to (79.1, 90.0)
- moved L6 47.6 mm to (79.1, 31.4)
- moved TP7 47.6 mm to (55.3, 77.5)
- moved U6 47.6 mm to (84.5, 35.9)
- moved U7 47.6 mm to (79.2, 36.5)
- moved ANT2 47.6 mm to (63.9, 89.1)
- moved C1 47.6 mm to (60.8, 64.1)
- moved C17 47.6 mm to (43.9, 69.9)
- moved C18 47.6 mm to (43.9, 72.4)
- moved C19 47.6 mm to (43.9, 74.9)
- moved C2 47.6 mm to (60.8, 66.1)
- moved C20 47.6 mm to (43.9, 77.4)
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Routing:
- added copper zone on In2.Cu, net +3V3
- added copper zone on B.Cu, net GND
- added copper zone on F.Cu, net GND
- added copper zone on In1.Cu, net GND
Other:
- board outline added: 50 x 100 mm

Commit message: PCB Layout
Parts:
- U5: moved to B.Cu
- moved SW1 114.2 mm to (151.3, 69.0), turned to 90 degrees
- moved L6 109.1 mm to (180.2, 72.2)
- moved SW2 107.3 mm to (144.8, 69.0), turned to 90 degrees
- moved SW6 102.7 mm to (138.3, 69.0), turned to 90 degrees
- moved U6 101.8 mm to (151.5, 112.5)
- moved U7 97.5 mm to (151.4, 102.0), turned to -90 degrees
- moved U1 96.6 mm to (143.2, 49.2), turned to -90 degrees
- moved SW5 95.2 mm to (131.8, 69.0), turned to 90 degrees
- moved ANT2 94.7 mm to (153.6, 58.7), turned to -90 degrees
- moved Q1 91.8 mm to (151.3, 107.7)
- moved U9 91.5 mm to (132.8, 58.8), turned to 90 degrees
- moved U8 89.8 mm to (151.2, 94.5)
- moved SW4 88.0 mm to (125.3, 69.0), turned to 90 degrees
- moved U3 87.5 mm to (142.8, 25.8), turned to 90 degrees
- moved U2 83.0 mm to (143.2, 58.9), turned to 180 degrees
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Other:
- board size 50 x 100 mm -> 40 x 82 mm

Commit message: PCB Work
Parts:
- removed C4: 0.1u, Capacitor_SMD:C_0402_1005Metric
- BT1: moved to B.Cu
- U5: moved to F.Cu
- moved L6 151.1 mm to (31.2, 47.1), turned to 90 degrees
- moved J3 132.7 mm to (24.5, 39.4), turned to 0 degrees
- moved U6 125.8 mm to (42.5, 49.6)
- moved SW2 120.9 mm to (24.5, 56.5)
- moved Q1 120.3 mm to (46.0, 49.6)
- moved SW1 119.4 mm to (32.5, 56.5)
- moved U7 117.8 mm to (44.0, 53.6), turned to 180 degrees
- moved U8 106.2 mm to (53.5, 53.0), turned to -90 degrees
- moved Y1 103.5 mm to (46.0, 43.0), turned to 0 degrees
- moved U9 100.5 mm to (34.7, 36.5), turned to 0 degrees
- moved U1 99.6 mm to (44.5, 36.5), turned to 180 degrees
- moved ANT2 97.8 mm to (62.5, 23.0), turned to 180 degrees
- moved U10 93.9 mm to (53.5, 43.0), turned to -90 degrees
- moved Y3 93.3 mm to (60.0, 29.2), turned to 0 degrees
- moved U5 91.9 mm to (26.9, 25.1), turned to 180 degrees
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Routing:
- net /OLED_VCC: track 0.00 -> 26.9 mm, vias 0 -> 2
- net Net-(U1-SPIQ): track 0.00 -> 16.8 mm, vias 0 -> 2
- net Net-(U1-SPIWP): track 0.00 -> 13.7 mm, vias 0 -> 2
- net Net-(U1-SPICS0): track 0.00 -> 11.7 mm, vias 0 -> 2
- net /OLED_MOSI: track 0.00 -> 8.58 mm
- net /OLED_SCK: track 0.00 -> 8.12 mm, vias 0 -> 2
- net /OLED_CS: track 0.00 -> 6.39 mm
- net /OLED_D/C: track 0.00 -> 6.33 mm, vias 0 -> 2
- net /VDD_SPI: track 0.00 -> 5.41 mm
- net Net-(U5-FB): track 0.00 -> 5.18 mm
- net Net-(D1-A): track 0.00 -> 4.99 mm
- net +SYS: track 0.00 -> 4.82 mm
- net Net-(U1-SPID): track 0.00 -> 4.77 mm
- net Net-(U1-SPICLK): track 0.00 -> 4.36 mm
- net Net-(U1-SPIHD): track 0.00 -> 4.34 mm
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- added copper zone on F.Cu, net +3V3
- added copper zone on F.Cu, net +SYS
- added copper zone on F.Cu, net Net-(U4-LX1)
- added copper zone on F.Cu, net Net-(U4-LX2)
Other:
- board size 40 x 82 mm -> 45 x 50 mm

Commit message: More changes
Parts:
- removed C27: 1u, Capacitor_SMD:C_0603_1608Metric
- moved R20 97.3 mm to (42.7, 49.9), turned to 180 degrees
- moved C24 82.4 mm to (56.4, 51.5)
- moved R2 75.2 mm to (56.9, 50.2), turned to 180 degrees
- moved R1 74.4 mm to (56.9, 49.1), turned to 180 degrees
- moved Q1 10.2 mm to (45.1, 59.8)
- moved U6 10.2 mm to (41.6, 59.8)
- moved U7 3.25 mm to (40.8, 54.1), turned to 90 degrees
- moved Y2 3.11 mm to (50.4, 33.3), turned to -90 degrees
- moved U8 2.49 mm to (52.5, 50.7)
- turned U3 to 90 degrees
Routing:
- net /USB_VBUS: track 0.00 -> 13.1 mm, vias 0 -> 2
- net /SCL: track 0.00 -> 5.01 mm
- net /SDA: track 0.00 -> 4.91 mm
- net Net-(J1-CC1): track 0.00 -> 3.84 mm
- net /D-: track 0.00 -> 3.01 mm
- net /D+: track 0.00 -> 2.84 mm
- net Net-(J1-CC2): track 0.00 -> 2.47 mm

Commit message: More PCB Work
Parts:
- removed C11, C15, C16: 0.1u, Capacitor_SMD:C_0402_1005Metric
- C14, C25, C26, C32, C33, C34, C53: moved to B.Cu
- moved C53 115.2 mm to (65.8, 26.2)
- moved C26 114.4 mm to (48.8, 24.6), turned to 90 degrees
- moved C52 113.0 mm to (65.3, 27.0), turned to 180 degrees
- moved C25 111.4 mm to (50.4, 24.6), turned to 90 degrees
- moved C43 108.7 mm to (53.3, 39.4), turned to 90 degrees
- moved C34 105.5 mm to (58.4, 37.5), turned to 180 degrees
- moved R39 103.5 mm to (48.0, 31.2), turned to -90 degrees
- moved C12 101.7 mm to (57.1, 35.5)
- moved C13 101.7 mm to (57.1, 37.5)
- moved C14 100.9 mm to (62.0, 37.5)
- moved C44 100.8 mm to (50.0, 40.4), turned to -90 degrees
- moved C36 100.5 mm to (50.0, 38.4), turned to -90 degrees
- moved R17 95.2 mm to (55.5, 33.5), turned to 180 degrees
- moved R33 90.0 mm to (56.2, 42.1), turned to 90 degrees
- moved L3 89.5 mm to (66.0, 25.3), turned to 90 degrees
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Connections:
- J2 pad 11: /OLED_RES -> /OLED_RST
Routing:
- net Net-(Q1A-S): track 0.00 -> 41.9 mm
- net /AP_EN: track 2.73 -> 30.1 mm, vias 0 -> 2
- net +3V3: track 1.64 -> 21.6 mm, vias 7 -> 16
- net /SCL: track 5.01 -> 23.3 mm, vias 0 -> 2
- net /SDA: track 4.91 -> 21.1 mm, vias 0 -> 2
- net Net-(ANT1-PadFEED): track 0.00 -> 15.0 mm
- net Net-(U1-XTAL_32K_P): track 0.00 -> 13.0 mm
- net Net-(J2-Pin_5): track 0.00 -> 11.4 mm, vias 0 -> 2
- net /ESP_RESET: track 0.00 -> 10.8 mm, vias 0 -> 2
- net Net-(U1-XTAL_32K_N): track 0.00 -> 9.82 mm
- net /OLED_RST: track 0.00 -> 7.00 mm, vias 0 -> 2
- net Net-(J2-Pin_9): track 0.00 -> 4.24 mm
- net Net-(U8-TMR): track 0.00 -> 4.11 mm
- net Net-(U1-LNA_IN): track 0.00 -> 3.56 mm
- net Net-(U2-RTC_O): track 0.00 -> 3.46 mm
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
Commit message: More PCB work
Parts:
- C47, C48, R26, Y2: moved to B.Cu
- moved D3 121.2 mm to (26.6, 33.0), turned to 180 degrees
- moved D2 118.9 mm to (26.6, 35.0), turned to 180 degrees
- moved C48 116.8 mm to (43.0, 33.2), turned to 90 degrees
- moved C47 113.4 mm to (46.0, 33.2), turned to 90 degrees
- moved R29 111.0 mm to (24.0, 33.0), turned to 180 degrees
- moved R28 108.2 mm to (24.0, 35.0), turned to 180 degrees
- moved R26 101.9 mm to (44.5, 33.6), turned to 180 degrees
- moved R19 95.3 mm to (37.8, 61.1)
- moved Y2 10.3 mm to (44.5, 35.5), turned to 180 degrees
Routing:
- net /GNSS_TP: track 0.00 -> 31.2 mm, vias 0 -> 2
- net /AP_EN: track 30.1 -> 0.00 mm, vias 2 -> 0
- net /GNSS_TXRDY: track 0.00 -> 20.9 mm, vias 0 -> 2
- net Net-(D3-K): track 0.00 -> 20.6 mm
- net /TPS_MODE: track 2.16 -> 22.4 mm, vias 0 -> 2
- net Net-(D2-K): track 0.00 -> 19.0 mm
- net Net-(U1-XTAL_32K_P): track 13.0 -> 7.87 mm, vias 0 -> 1
- net +3V3: track 21.6 -> 25.5 mm, vias 16 -> 18
- net Net-(D3-A): track 0.00 -> 1.30 mm
- net Net-(D2-A): track 0.00 -> 1.30 mm
- net Net-(U1-XTAL_32K_N): track 9.82 -> 8.66 mm, vias 0 -> 1
- net GND: vias 32 -> 30

Commit message: More PCB work
Parts:
- C10, C9, L4: moved to B.Cu
- moved C42 108.7 mm to (47.4, 41.7), turned to -90 degrees
- moved C46 105.8 mm to (42.9, 44.2), turned to -90 degrees
- moved C35 105.1 mm to (52.1, 46.6), turned to 90 degrees
- moved C45 102.0 mm to (46.3, 44.2), turned to -90 degrees
- moved C10 101.4 mm to (46.6, 39.5), turned to 180 degrees
- moved C9 100.3 mm to (48.5, 37.5)
- moved C3 96.6 mm to (39.4, 52.1), turned to 180 degrees
- moved C19 94.5 mm to (48.7, 42.2), turned to -90 degrees
- moved C22 89.9 mm to (51.0, 53.7)
- moved R25 89.6 mm to (39.9, 50.5), turned to -90 degrees
- moved R24 88.9 mm to (38.8, 50.5), turned to -90 degrees
- moved R30 87.5 mm to (43.7, 48.5), turned to -90 degrees
- moved R27 86.1 mm to (46.3, 42.2), turned to 90 degrees
- moved L4 85.7 mm to (48.1, 39.0), turned to -90 degrees
- moved R22 82.4 mm to (44.9, 49.9), turned to -90 degrees
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Connections:
- BT1 pad P2: Net-(Q1A-S) -> (no net)
Routing:
- net /SDA: track 21.1 -> 47.2 mm, vias 2 -> 4
- net /SCL: track 23.3 -> 48.4 mm, vias 2 -> 4
- net /TPS_MODE: track 22.4 -> 45.5 mm
- net Net-(Q1A-S): track 41.9 -> 26.6 mm, vias 0 -> 3
- net Net-(Q1B-S): track 0.00 -> 14.5 mm, vias 0 -> 2
- net Net-(BT1--): track 0.00 -> 13.9 mm, vias 0 -> 2
- net Net-(U7-GPOUT): track 0.00 -> 8.78 mm, vias 0 -> 2
- net Net-(Q1B-G): track 0.00 -> 6.59 mm, vias 0 -> 2
- net Net-(U1-XTAL_N): track 0.00 -> 6.25 mm
- net GND: track 0.00 -> 4.49 mm, vias 30 -> 40
- net Net-(U8-TS): track 0.00 -> 3.93 mm
- net Net-(U6-PACK): track 0.00 -> 3.76 mm
- net Net-(U7-VDD): track 0.00 -> 3.69 mm
- net Net-(U7-BIN): track 0.00 -> 3.39 mm
- net Net-(U6-VDD): track 0.00 -> 3.15 mm
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- added copper zone on B.Cu, net +SYS
- added copper zone on F.Cu, net BAT
- added copper zone on F.Cu, net Net-(C9-Pad1)
- added copper zone on F.Cu, net Net-(Q1A-D-Pad6)
- added copper zone on F.Cu, net Net-(Q1B-S)
