File: ESPWatchS3.kicad_pcb (KiCad board)
At the start: 6 copper layers, 80 x 80 mm, 109 parts, among them J1 OLED, J2 USB, J3 UART0, U1 ESP32-S3R8, U10 BD48KxxG, U2 EVA-M8Q-0, U3 BME280, U4 IS25LP128F-JKLE, U5 BQ27441-G1A, U6 BQ24075RGTR, U7 TPS631000DRLR, U8 AP3012, U9 NJG1143UA2-TE1, Y1 40MHz, Y2 32.768kHz, Y3 32.768kHz

Commit message: Initial PCB work for V1.0
Parts:
- C17, D1, L3, L4, R20, R21, R22, U10, U5, U6, U7, U8: moved to B.Cu
- moved ANT1 131.5 mm to (21.0, 40.0), turned to -90 degrees
- moved L4 122.9 mm to (36.4, 36.3), turned to -90 degrees
- moved BT1 120.4 mm to (32.0, 36.5), turned to 180 degrees
- moved R20 114.7 mm to (38.0, 24.5), turned to 90 degrees
- moved R21 111.3 mm to (41.5, 24.5), turned to 90 degrees
- moved R22 97.7 mm to (45.5, 31.5), turned to -90 degrees
- moved J2 97.3 mm to (40.0, 23.5), turned to 180 degrees
- moved S2 96.0 mm to (27.5, 52.5), turned to -45 degrees
- moved C17 95.6 mm to (36.6, 32.3), turned to 180 degrees
- moved Y1 95.0 mm to (43.0, 36.5), turned to 90 degrees
- moved U4 94.6 mm to (51.0, 44.5), turned to 180 degrees
- moved U7 94.3 mm to (40.0, 36.3)
- moved U1 94.1 mm to (40.0, 42.0), turned to 90 degrees
- moved S1 94.1 mm to (27.5, 27.5), turned to -135 degrees
- moved U2 94.0 mm to (51.0, 36.0), turned to -90 degrees
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Routing:
- net /USB_VBUS: track 0.00 -> 12.5 mm, vias 0 -> 2
- net Net-(J2-CC2): track 0.00 -> 2.27 mm, vias 0 -> 1
- net Net-(J2-CC1): track 0.00 -> 2.27 mm, vias 0 -> 1
- added copper zone on In2.Cu, net +3V3
- added copper zone on B.Cu, net Net-(U7-LX1)
- added copper zone on B.Cu, net Net-(U7-LX2)
Other:
- board size 80 x 80 mm -> 40 x 40 mm

Commit message: PCB Work
Parts:
- added H1: MountingHole, MountingHole:MountingHole_2.2mm_M2, F.Cu at (24.0, 33.0)
- added H2: MountingHole, MountingHole:MountingHole_2.2mm_M2, F.Cu at (24.0, 47.0)
- added H3: MountingHole, MountingHole:MountingHole_2.2mm_M2, F.Cu at (56.0, 33.0)
- added H4: MountingHole, MountingHole:MountingHole_2.2mm_M2, F.Cu at (56.0, 47.0)
- C18, C26, C27, C5, L5: moved to B.Cu
- moved R26 124.5 mm to (31.9, 43.4), turned to 180 degrees
- moved R11 117.2 mm to (32.4, 26.6)
- moved Y2 115.5 mm to (42.4, 49.7)
- moved L5 112.6 mm to (31.7, 42.3), turned to 90 degrees
- moved C34 105.6 mm to (32.4, 27.6)
- moved C27 104.9 mm to (30.6, 42.3), turned to -90 degrees
- moved Y3 104.1 mm to (54.4, 37.5), turned to -90 degrees
- moved FL1 103.7 mm to (55.1, 43.4)
- moved C18 103.1 mm to (29.5, 42.3), turned to -90 degrees
- moved C26 102.9 mm to (32.8, 42.3), turned to 90 degrees
- moved C5 101.5 mm to (28.4, 42.3), turned to -90 degrees
- moved C32 100.5 mm to (34.7, 38.4), turned to 90 degrees
- moved C16 99.1 mm to (33.5, 38.4), turned to 90 degrees
- moved C22 94.5 mm to (38.0, 48.8), turned to -90 degrees
- moved C23 92.5 mm to (39.9, 38.3), turned to 90 degrees
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Routing:
- net GND: track 0.00 -> 30.5 mm, vias 0 -> 37
- net /ESP_U0RX: track 0.00 -> 16.1 mm, vias 0 -> 2
- net +3V3: track 0.00 -> 14.4 mm, vias 0 -> 5
- net Net-(U1-SPIQ): track 0.00 -> 11.9 mm, vias 0 -> 2
- net /OLED_MOSI: track 0.00 -> 10.4 mm
- net Net-(U1-SPICS0): track 0.00 -> 10.00 mm, vias 0 -> 2
- net /OLED_SCK: track 0.00 -> 9.79 mm, vias 0 -> 2
- net Net-(U1-U0TXD): track 0.00 -> 9.63 mm, vias 0 -> 2
- net Net-(U1-SPIWP): track 0.00 -> 9.40 mm, vias 0 -> 2
- net /OLED_D/C: track 0.00 -> 8.46 mm, vias 0 -> 2
- net /OLED_RST: track 0.00 -> 7.72 mm, vias 0 -> 2
- net /OLED_CS: track 0.00 -> 7.41 mm
- net /ESP_BOOT: track 0.00 -> 7.40 mm
- net Net-(U1-XTAL_32K_N): track 0.00 -> 6.87 mm
- net Net-(U2-RTC_O): track 0.00 -> 6.68 mm
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- added copper zone on In3.Cu, net +3V3
- removed copper zone on In2.Cu, net +3V3
- removed copper zone on B.Cu, net GND
- removed copper zone on F.Cu, net GND

Commit message: PCB Work
Parts:
- R18, R19: moved to B.Cu
- moved R18 117.4 mm to (35.8, 39.8), turned to -90 degrees
- moved R24 116.6 mm to (35.9, 37.3), turned to -90 degrees
- moved R19 116.1 mm to (36.9, 39.8), turned to -90 degrees
- moved C37 101.7 mm to (36.3, 35.7)
- moved R14 100.3 mm to (49.5, 41.0)
- moved C38 99.8 mm to (38.2, 35.7), turned to 180 degrees
- moved C29 97.9 mm to (37.4, 32.9), turned to 180 degrees
- moved C28 97.8 mm to (37.4, 31.5), turned to 180 degrees
- moved L6 88.1 mm to (56.2, 43.5)
- moved C45 87.6 mm to (53.6, 42.0), turned to 180 degrees
- moved C44 86.0 mm to (55.4, 40.5)
- moved FL1 3.51 mm to (53.1, 40.5), turned to 180 degrees
- moved U9 0.49 mm to (55.5, 42.0), turned to 180 degrees
- moved Y1 0.39 mm to (37.8, 37.4), turned to -90 degrees
- moved C17 0.05 mm to (36.5, 32.3)
Routing:
- net /SDA: track 0.00 -> 16.7 mm, vias 0 -> 2
- net /SCL: track 0.00 -> 16.1 mm, vias 0 -> 2
- net GND: track 30.5 -> 40.9 mm, vias 37 -> 43
- net Net-(U2-ANT_OFF): track 0.00 -> 10.2 mm, vias 0 -> 2
- net +3V3: track 14.4 -> 23.4 mm, vias 5 -> 6
- net Net-(U1-XTAL_N): track 0.00 -> 5.38 mm
- net Net-(FL1-OUTPUT): track 0.00 -> 3.24 mm
- net Net-(C37-Pad1): track 0.00 -> 3.20 mm
- net Net-(U1-XTAL_P): track 0.00 -> 2.67 mm
- net Net-(U1-U0TXD): track 9.63 -> 12.1 mm
- net /ESP_U0RX: track 16.1 -> 17.9 mm
- net Net-(ANT2-FEED): track 0.00 -> 1.77 mm
- net Net-(U9-RFIN): track 0.00 -> 1.53 mm
- net Net-(FL1-INPUT): track 0.00 -> 1.22 mm
- net Net-(U9-RFOUT): track 0.00 -> 1.01 mm

Commit message: Significant PCB work
Parts:
- C10, C12, C15, C3, C8, R1, R2, R25: moved to B.Cu
- moved C8 128.6 mm to (32.2, 53.0), turned to -90 degrees
- moved C9 127.0 mm to (33.0, 49.7), turned to 90 degrees
- moved R32 120.5 mm to (35.4, 50.2), turned to 90 degrees
- moved R25 119.9 mm to (34.0, 57.9), turned to 90 degrees
- moved R17 118.9 mm to (31.1, 49.8)
- moved C10 112.5 mm to (47.8, 53.0), turned to -90 degrees
- moved R1 111.6 mm to (34.0, 55.5), turned to 90 degrees
- moved R2 106.2 mm to (39.9, 59.4), turned to 180 degrees
- moved C31 104.2 mm to (31.1, 48.7)
- moved C39 99.2 mm to (39.2, 48.8), turned to -90 degrees
- moved C19 99.0 mm to (34.4, 50.2), turned to 90 degrees
- moved C40 97.9 mm to (40.4, 48.8), turned to -90 degrees
- moved C3 97.8 mm to (35.2, 54.0), turned to 90 degrees
- moved C12 94.2 mm to (36.3, 54.0), turned to 90 degrees
- moved C15 91.8 mm to (44.9, 56.0), turned to 180 degrees
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Routing:
- net /D-: track 0.00 -> 31.7 mm, vias 0 -> 2
- net /D+: track 0.00 -> 31.4 mm, vias 0 -> 2
- net /OLED_VCC: track 0.00 -> 29.2 mm, vias 0 -> 3
- net /GNSS_RX: track 0.00 -> 26.4 mm, vias 0 -> 2
- net /GNSS_TX: track 0.00 -> 22.6 mm, vias 0 -> 2
- net /GNSS_TP: track 0.00 -> 15.9 mm, vias 0 -> 2
- net GND: track 40.9 -> 29.0 mm, vias 43 -> 56
- net /SDA: track 16.7 -> 25.7 mm, vias 2 -> 3
- net /ESP_RESET: track 5.79 -> 13.6 mm, vias 0 -> 2
- net /SCL: track 16.1 -> 23.3 mm, vias 2 -> 3
- net Net-(U8-FB): track 0.00 -> 6.35 mm
- net /USB_VBUS: track 12.6 -> 6.64 mm
- net Net-(J1-Pin_3): track 0.00 -> 4.67 mm
- net Net-(J1-Pin_9): track 0.00 -> 4.61 mm
- net +3V3: track 23.4 -> 27.8 mm, vias 6 -> 8
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- added copper zone on B.Cu, net +SYS
- added copper zone on B.Cu, net /OLED_VCC
- added copper zone on B.Cu, net GND
- added copper zone on F.Cu, net GND
- added copper zone on B.Cu, net Net-(D1-A)

Commit message: More PCB work
Parts:
- moved L1 122.6 mm to (22.2, 43.4), turned to 90 degrees
- moved C41 114.3 mm to (23.7, 43.9)
- moved R6 113.2 mm to (34.8, 48.7)
- moved L2 112.1 mm to (32.2, 40.9)
- moved C42 110.9 mm to (30.6, 40.4), turned to 90 degrees
- moved C43 107.5 mm to (33.9, 40.4), turned to 90 degrees
- moved BT1 2.00 mm to (29.9, 34.5)
- moved H1 1.00 mm to (23.0, 33.0)
- moved H2 1.00 mm to (23.0, 47.0)
- moved H3 1.00 mm to (57.0, 33.0)
- moved H4 1.00 mm to (57.0, 47.0)
Routing:
- net /GNSS_TXRDY: track 0.00 -> 17.6 mm, vias 0 -> 2
- net Net-(ANT1-PadFEED): track 0.00 -> 12.2 mm
- net /AP_EN: track 2.15 -> 13.1 mm, vias 0 -> 1
- net /ESP_BOOT: track 7.40 -> 9.80 mm
- net Net-(U1-LNA_IN): track 0.00 -> 2.38 mm
- net /ESP_RESET: track 13.6 -> 15.1 mm
- net GND: track 29.0 -> 27.7 mm, vias 56 -> 62
- net Net-(C41-Pad1): track 0.00 -> 1.03 mm
- net +3V3: vias 8 -> 11

Commit message: Even more!
Parts:
- C13, C14, R10, R15, R16, R27, R28, R29, R8: moved to B.Cu
- moved R28 126.4 mm to (29.0, 29.8), turned to 180 degrees
- moved TH1 124.4 mm to (34.5, 35.9), turned to -90 degrees
- moved R27 122.9 mm to (32.5, 26.6), turned to 90 degrees
- moved R29 122.0 mm to (33.5, 26.6), turned to 90 degrees
- moved R16 120.2 mm to (29.4, 31.7), turned to 90 degrees
- moved R15 118.8 mm to (30.8, 37.0), turned to 180 degrees
- moved R5 115.9 mm to (30.7, 30.2), turned to -90 degrees
- moved R4 114.3 mm to (32.5, 32.0), turned to 180 degrees
- moved R8 109.8 mm to (37.4, 46.1)
- moved R10 109.5 mm to (37.4, 47.2)
- moved C13 103.8 mm to (25.9, 32.8), turned to 90 degrees
- moved C14 103.8 mm to (25.9, 34.8), turned to -90 degrees
- moved U5 34.4 mm to (29.1, 34.6), turned to 0 degrees
- moved R22 27.7 mm to (32.8, 34.6), turned to -90 degrees
- moved U6 25.3 mm to (32.2, 30.5), turned to 180 degrees
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Routing:
- net /CHG_EN2: track 0.00 -> 25.5 mm, vias 0 -> 3
- net /CHG_EN1: track 0.00 -> 25.3 mm, vias 0 -> 3
- net /CHG_PWRGD: track 0.00 -> 25.3 mm, vias 0 -> 3
- net /CHG_CHG: track 0.00 -> 24.9 mm, vias 0 -> 3
- net Net-(BT1-+): track 0.00 -> 19.6 mm, vias 0 -> 1
- net GND: track 27.7 -> 39.7 mm, vias 62 -> 73
- net /USB_VBUS: track 6.64 -> 14.9 mm
- net Net-(U5-BIN): track 0.00 -> 8.00 mm, vias 0 -> 2
- net Net-(U6-TS): track 0.00 -> 7.31 mm, vias 0 -> 1
- net BAT: track 0.00 -> 6.12 mm, vias 0 -> 2
- net +3V3: track 27.8 -> 32.1 mm, vias 11 -> 13
- net /ESP_U0TX: track 3.49 -> 6.27 mm, vias 0 -> 2
- net Net-(U6-ISET): track 0.00 -> 2.42 mm, vias 0 -> 2
- net Net-(U6-TMR): track 0.00 -> 2.13 mm, vias 0 -> 2
- net /ESP_U0RX: track 17.9 -> 19.8 mm
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- added copper zone on B.Cu, net BAT

Commit message: Even more
Parts:
- C1, C2, C24, C25, R26: moved to B.Cu
- C18, C26, C27, C5, L5: moved to F.Cu
- moved C2 113.8 mm to (46.0, 42.9), turned to 90 degrees
- moved C1 103.3 mm to (50.6, 42.6), turned to 90 degrees
- moved C24 91.7 mm to (44.8, 43.4), turned to 90 degrees
- moved C25 84.1 mm to (52.1, 43.4), turned to 90 degrees
- moved L4 42.6 mm to (48.2, 46.7), turned to 0 degrees
- moved U7 37.6 mm to (48.2, 43.1), turned to 90 degrees
- moved R14 0.70 mm to (50.2, 41.0), turned to 90 degrees
- moved C5 0.53 mm to (28.9, 42.3), turned to 90 degrees
- moved C18 0.48 mm to (29.9, 42.3), turned to 90 degrees
- moved C27 0.48 mm to (31.1, 42.3), turned to 90 degrees
- moved L5 0.43 mm to (32.1, 42.3), turned to -90 degrees
- moved C26 0.39 mm to (33.1, 42.3), turned to -90 degrees
- moved C42 0.15 mm to (31.8, 39.2)
- moved L2 0.10 mm to (32.2, 40.8)
- moved C43 0.08 mm to (33.9, 40.3)
Routing:
- net GND: track 39.7 -> 41.7 mm, vias 73 -> 76
- net Net-(U1-U0TXD): track 12.3 -> 10.8 mm
- net Net-(U2-ANT_OFF): track 10.2 -> 9.45 mm
- net Net-(C26-Pad1): track 4.09 -> 3.49 mm, vias 1 -> 0
- net +3V3: track 32.1 -> 32.6 mm, vias 13 -> 17
- added copper zone on B.Cu, net +3V3

Commit message: Routing continues
Parts:
- R30, R31: moved to B.Cu
- moved R30 106.0 mm to (49.7, 43.2), turned to 90 degrees
- moved R31 105.7 mm to (49.7, 41.2), turned to 90 degrees
- moved C1 0.85 mm to (51.2, 43.2)
- moved C25 0.76 mm to (52.8, 43.8)
- moved R16 0.71 mm to (28.9, 32.2), turned to 180 degrees
- moved L4 0.57 mm to (47.9, 47.1)
- moved U7 0.57 mm to (47.9, 43.5)
- moved C2 0.57 mm to (45.7, 43.3)
- moved C24 0.48 mm to (44.4, 43.7)
- moved C21 0.46 mm to (46.5, 48.9)
- moved R14 0.35 mm to (50.5, 41.0)
Routing:
- net Net-(U7-FB): track 0.00 -> 2.04 mm
- net Net-(U1-SPIWP): track 9.26 -> 11.0 mm
- net GND: track 41.7 -> 43.0 mm, vias 76 -> 79
- net Net-(U1-SPIQ): track 11.9 -> 12.7 mm
- net Net-(U5-BIN): track 8.00 -> 7.26 mm
- net /CHG_CHG: track 24.9 -> 25.4 mm
- net +SYS: vias 0 -> 13
- added copper zone on In2.Cu, net +SYS
