File: ESPWatchS3.kicad_pcb (KiCad board)
At the start: 6 copper layers, 34 x 40 mm, 126 parts, among them J1 USB, J2 LCD, J3 UART0, Q1 DMC2053UVT, U1 ESP32-S3R8, U10 SN74LV1T34DCK, U11 AP3036B, U2 IS25LP128F-JKLE, U3 MIA-M10Q-00B, U4 ICM-42688-P, U5 BMP390, U6 BQ24075RGTR, U7 BQ27441-G1A, U8 TPS631000DRLR, U9 BD48xxFVE, Y1 40MHz, Y2 32.768kHz, Y3 32.768kHz

Commit message: Routing work
Parts:
- ANT2: value 1575AT43A0040E -> W3011A; footprint WatchParts:1575AT43A0040E -> WatchParts:ANTENNA_W3011A
- C14, C15, C19, C22, C24, C26, C4, H3, L5, R22, R23, U9: moved to B.Cu
- C47: value DNF -> 3.3p
- U6: moved to F.Cu
- moved U4 104.2 mm to (79.7, 34.1)
- moved C1 80.8 mm to (55.9, 45.3)
- moved C23 78.0 mm to (55.1, 50.5)
- moved D1 77.0 mm to (52.0, 55.0), turned to 90 degrees
- moved C10 74.3 mm to (50.0, 53.8)
- moved C11 74.0 mm to (50.0, 54.9)
- moved C3 73.3 mm to (43.8, 50.9), turned to -90 degrees
- moved C12 72.7 mm to (51.7, 45.6), turned to 180 degrees
- moved C13 72.7 mm to (48.0, 47.0), turned to 90 degrees
- moved C7 71.6 mm to (51.4, 30.4), turned to -90 degrees
- moved C30 70.7 mm to (56.8, 28.0)
- moved C18 69.6 mm to (51.3, 38.1)
- moved C9 68.5 mm to (48.2, 34.8), turned to 180 degrees
- moved R31 67.5 mm to (42.5, 54.4), turned to -90 degrees
- moved C29 66.6 mm to (52.5, 30.4), turned to -90 degrees
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Connections:
- C47 pad 1: Net-(ANT2-FEED) -> Net-(ANT2-PadFEED)
- L6 pad 2: Net-(ANT2-FEED) -> Net-(ANT2-PadFEED)
Routing:
- net /USB_VBUS: track 0.00 -> 28.2 mm, vias 0 -> 3
- net Net-(BT1-+): track 0.00 -> 19.7 mm, vias 0 -> 2
- net GND: track 0.00 -> 18.7 mm, vias 0 -> 77
- net /LCD_TE: track 0.00 -> 16.0 mm, vias 0 -> 3
- net /LCD_DC: track 0.00 -> 13.3 mm, vias 0 -> 2
- net Net-(U1-SPIQ): track 0.00 -> 13.1 mm, vias 0 -> 2
- net Net-(U1-SPICS0): track 0.00 -> 12.5 mm, vias 0 -> 2
- net +3V3: track 0.00 -> 12.4 mm, vias 0 -> 15
- net Net-(ANT1-PadFEED): track 0.00 -> 9.64 mm
- net Net-(U1-SPIWP): track 0.00 -> 9.60 mm, vias 0 -> 2
- net /VDD_SPI: track 0.00 -> 8.27 mm
- net /GNSS_TXRDY: track 0.00 -> 8.11 mm, vias 0 -> 2
- net Net-(D1-K): track 0.00 -> 8.02 mm, vias 0 -> 2
- net /GNSS_TP: track 0.00 -> 6.27 mm
- net Net-(U1-SPICLK): track 0.00 -> 5.84 mm
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- added copper zone on F.Cu, net +3V3
- added copper zone on F.Cu, net +SYS
- added copper zone on F.Cu, net BAT
- added copper zone on F.Cu, net Net-(U8-LX1)
- added copper zone on F.Cu, net Net-(U8-LX2)
- removed copper zone on F.Cu, net Net-(ANT2-FEED)

Commit message: Layout continues
Parts:
- C21, C35, D2, Q1, R20, R4, R7, R8, R9, U10, Y3: moved to B.Cu
- U9: moved to F.Cu
- moved D2 75.5 mm to (50.5, 48.5)
- moved R9 56.9 mm to (57.2, 49.9), turned to 90 degrees
- moved R8 52.7 mm to (52.8, 49.0), turned to -90 degrees
- moved R7 49.0 mm to (49.1, 46.1), turned to -90 degrees
- moved C33 46.9 mm to (32.6, 31.1), turned to -90 degrees
- moved C21 46.9 mm to (30.0, 31.6), turned to 180 degrees
- moved C17 45.8 mm to (28.1, 30.4), turned to -90 degrees
- moved Q1 44.5 mm to (55.0, 48.5)
- moved Y3 42.2 mm to (54.7, 25.1), turned to 180 degrees
- moved C35 41.4 mm to (30.1, 22.6), turned to 180 degrees
- moved R4 39.9 mm to (30.1, 23.6)
- moved U4 36.3 mm to (44.0, 41.1)
- moved U9 36.1 mm to (29.9, 29.4), turned to 180 degrees
- moved R29 34.0 mm to (36.0, 26.1), turned to 90 degrees
- moved J3 34.0 mm to (33.6, 26.9)
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Routing:
- net +SYS: track 0.00 -> 56.0 mm, vias 0 -> 3
- net /FUEL_GPO: track 0.81 -> 25.5 mm, vias 1 -> 2
- net Net-(J3-Pin_6): track 0.00 -> 13.4 mm, vias 0 -> 2
- net /ESP_RESET: track 0.00 -> 13.3 mm, vias 0 -> 2
- net /ESP_BOOT: track 0.00 -> 11.4 mm
- net Net-(U1-U0TXD): track 0.00 -> 11.4 mm, vias 0 -> 2
- net GND: track 18.7 -> 30.0 mm, vias 77 -> 82
- net /PWR_BTN: track 0.00 -> 10.7 mm, vias 0 -> 1
- net Net-(U3-RTC_I): track 0.00 -> 9.14 mm, vias 0 -> 1
- net Net-(U3-RTC_O): track 0.00 -> 6.31 mm, vias 0 -> 1
- net /SMPS_EN2: track 0.00 -> 5.27 mm, vias 0 -> 1
- net Net-(U10-A): track 0.00 -> 4.94 mm
- net Net-(C35-Pad2): track 0.00 -> 3.04 mm, vias 0 -> 1
- net +3V3: track 12.4 -> 15.1 mm, vias 15 -> 19
- net Net-(Q1A-G): track 0.00 -> 2.55 mm
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
Commit message: More of the same
Parts:
- R5: moved to B.Cu
- moved C8 68.8 mm to (46.9, 41.4)
- moved C31 62.1 mm to (46.9, 42.5)
- moved C42 59.3 mm to (48.0, 36.4), turned to 90 degrees
- moved C32 58.7 mm to (43.5, 43.7), turned to -90 degrees
- moved R5 57.7 mm to (55.9, 46.0), turned to 90 degrees
- moved C41 53.9 mm to (42.4, 36.6), turned to 180 degrees
- moved L2 46.5 mm to (38.4, 43.7), turned to 180 degrees
- moved R3 40.6 mm to (37.1, 33.9), turned to 180 degrees
- moved R2 40.4 mm to (37.1, 32.9), turned to 180 degrees
- moved R32 39.6 mm to (45.5, 38.4)
- moved R14 37.5 mm to (33.7, 31.1), turned to -90 degrees
- moved D3 36.3 mm to (34.6, 48.1), turned to 180 degrees
- moved U11 35.9 mm to (38.4, 47.2), turned to 180 degrees
- moved U5 20.9 mm to (18.2, 42.8)
- moved C26 5.27 mm to (45.5, 34.1), turned to 90 degrees
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Connections:
- S3 pad 3: unconnected-(S3-Pad3) -> (no net)
- S3 pad 4: unconnected-(S3-Pad3) -> (no net)
Routing:
- net /CHG_EN1: track 0.00 -> 29.4 mm, vias 0 -> 2
- net /CHG_EN2: track 0.00 -> 28.6 mm, vias 0 -> 2
- net /IMU_INT2: track 0.00 -> 18.4 mm, vias 0 -> 2
- net /IMU_INT1: track 0.00 -> 13.4 mm, vias 0 -> 2
- net GND: track 30.0 -> 40.6 mm, vias 82 -> 85
- net Net-(U1-XTAL_32K_N): track 0.00 -> 8.49 mm
- net +3V3: track 15.1 -> 22.3 mm, vias 19 -> 27
- net Net-(U1-XTAL_32K_P): track 0.00 -> 6.65 mm
- net /FUEL_GPO: track 25.5 -> 27.7 mm
- net /SMPS_EN2: track 5.27 -> 6.66 mm

Commit message: Just 50 nets left!
Parts:
- moved C6 78.9 mm to (57.1, 37.9), turned to 180 degrees
- moved C16 77.5 mm to (58.7, 37.6), turned to 90 degrees
- moved C27 62.0 mm to (43.2, 46.0)
- moved C28 60.5 mm to (42.0, 47.0)
- moved R13 59.5 mm to (59.9, 37.6), turned to 90 degrees
- moved R30 52.6 mm to (59.6, 44.1), turned to -90 degrees
- moved R15 34.0 mm to (38.0, 31.1), turned to -90 degrees
- moved R25 29.4 mm to (36.4, 33.4), turned to 90 degrees
- moved R24 28.3 mm to (35.3, 33.4), turned to 90 degrees
- moved D3 23.0 mm to (57.2, 43.6)
- moved U5 23.0 mm to (41.0, 45.2)
- moved U11 21.3 mm to (58.7, 40.7), turned to -90 degrees
- moved L2 17.1 mm to (55.2, 40.7), turned to -90 degrees
- moved C26 1.68 mm to (43.9, 33.6), turned to 180 degrees
- moved C15 1.58 mm to (45.9, 33.6), turned to 0 degrees
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Connections:
- J1 pad S1: unconnected-(J1-SHIELD-PadS1) -> (no net)
- S1 pad 3: unconnected-(S1-Pad3) -> (no net)
- S1 pad 4: unconnected-(S1-Pad3) -> (no net)
- S2 pad 3: unconnected-(S2-Pad3) -> (no net)
- S2 pad 4: unconnected-(S2-Pad3) -> (no net)
- S4 pad 3: unconnected-(S4-Pad3) -> (no net)
- S4 pad 4: unconnected-(S4-Pad3) -> (no net)
Routing:
- net /SDA: track 2.65 -> 58.6 mm, vias 1 -> 6
- net /SCL: track 1.92 -> 56.0 mm, vias 1 -> 5
- net /D-: track 3.58 -> 21.6 mm, vias 0 -> 2
- net /D+: track 3.56 -> 20.9 mm, vias 0 -> 2
- net +3V3: track 22.3 -> 36.8 mm, vias 27 -> 33
- net Net-(J2-Pin_2): track 0.00 -> 14.3 mm, vias 0 -> 1
- net Net-(D3-A): track 0.00 -> 14.1 mm, vias 0 -> 1
- net GND: track 40.6 -> 48.7 mm, vias 85 -> 95
- net /GNSS_RX: track 0.00 -> 3.85 mm, vias 0 -> 1
- net Net-(D3-K): track 0.00 -> 3.82 mm
- net Net-(U1-GPIO3): track 0.00 -> 2.71 mm
- net Net-(U11-SW): track 0.00 -> 2.66 mm
- net /GNSS_TX: track 0.00 -> 2.27 mm, vias 0 -> 1
- net /LCD_BL: track 1.14 -> 2.69 mm
- net Net-(J1-CC2): track 2.19 -> 1.22 mm
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
Commit message: PCB Fully Routed
Parts:
- R19: moved to B.Cu
- TP1, TP2, TP3, TP4, TP5, TP6, TP7, TP8: footprint TestPoint:TestPoint_Pad_D1.0mm -> WatchParts:TestPoint_Pad_D0.5mm
- moved C37 78.3 mm to (59.5, 55.9), turned to 90 degrees
- moved C5 77.0 mm to (49.2, 52.3), turned to -90 degrees
- moved TP1 71.6 mm to (52.0, 41.2)
- moved C25 71.1 mm to (51.6, 45.6), turned to 180 degrees
- moved TP7 70.5 mm to (59.1, 31.9)
- moved TP8 70.2 mm to (59.0, 35.4)
- moved C36 70.1 mm to (58.5, 28.8), turned to 90 degrees
- moved TP6 65.6 mm to (52.0, 42.5)
- moved TP2 62.0 mm to (42.2, 50.4)
- moved R10 59.8 mm to (59.5, 28.8), turned to -90 degrees
- moved R6 58.7 mm to (58.8, 45.8)
- moved R11 58.4 mm to (58.4, 55.9), turned to -90 degrees
- moved TP4 50.5 mm to (33.9, 44.2)
- moved C38 49.2 mm to (31.4, 48.7), turned to 180 degrees
- moved TP3 48.3 mm to (31.8, 44.2)
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Routing:
- net /USER_BTN3: track 0.00 -> 50.1 mm, vias 0 -> 4
- net Net-(C35-Pad2): track 3.04 -> 46.8 mm
- net /SMPS_MODE: track 0.00 -> 33.3 mm, vias 0 -> 3
- net /SDA: track 58.6 -> 89.3 mm, vias 6 -> 9
- net /SMPS_EN1: track 1.36 -> 31.0 mm, vias 0 -> 2
- net /SCL: track 56.0 -> 84.6 mm, vias 5 -> 8
- net /LCD_BL: track 2.69 -> 31.2 mm, vias 1 -> 2
- net /USER_BTN1: track 0.00 -> 26.8 mm, vias 0 -> 2
- net /USER_BTN2: track 0.00 -> 24.1 mm, vias 0 -> 2
- net /GNSS_TX: track 2.27 -> 14.5 mm, vias 1 -> 2
- net Net-(U6-TS): track 0.00 -> 11.7 mm, vias 0 -> 2
- net /GNSS_RX: track 3.85 -> 15.1 mm, vias 1 -> 2
- net /ESP_RESET: track 13.3 -> 23.6 mm, vias 2 -> 3
- net Net-(U3-RESET_N): track 0.00 -> 9.21 mm, vias 0 -> 2
- net GND: track 48.7 -> 57.7 mm, vias 95 -> 105
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
Commit message: Cleanup work, silkscreen, file exports
Parts:
- ANT1: value W3008G -> W3008C; footprint WatchParts:ANTENNA_W3008 -> WatchParts:ANTENNA_W3008C
- J3: value UART0 -> UART
- TP7: value GNSS Reset -> G_RES
- moved TP3 6.41 mm to (35.0, 38.7)
- moved TP4 6.17 mm to (36.6, 38.7)
- moved C43 1.71 mm to (38.8, 25.1)
- moved C45 1.50 mm to (38.8, 19.9), turned to 90 degrees
- moved C44 1.10 mm to (37.7, 25.1), turned to 90 degrees
- moved L3 0.85 mm to (37.3, 20.3)
- moved L4 0.84 mm to (38.2, 26.6)
- moved Y3 0.50 mm to (54.7, 25.6)
Routing:
- net /SDA: track 89.3 -> 83.5 mm
- net /SCL: track 84.6 -> 79.2 mm
- net Net-(U1-LNA_IN): track 2.45 -> 3.51 mm
- net Net-(U3-RTC_O): track 6.31 -> 5.81 mm
- net Net-(U3-RTC_I): track 9.14 -> 8.64 mm
- net GND: vias 105 -> 221
Other:
- board text added: "BMP"
- board text added: "ESPWatchS3 V1.0 Design By: Sam Bach"
- board text added: "Flash"
- board text added: "GNSS"
- board text added: "IMU"
- board text added: "MCU"
- board text added: "WiFi"

Commit message: Update production files
Parts:
- C29, C30, C7: moved to B.Cu
- L2: footprint Inductor_SMD:L_1210_3225Metric -> WatchParts:IND_VLS201612CX-220M-1
- TP7: value G_RES -> UBX_RST
- moved L2 0.55 mm to (55.8, 40.7)
- moved C6 0.54 mm to (57.6, 37.6), turned to 90 degrees
- moved C29 0.35 mm to (52.5, 30.8)
- moved C7 0.35 mm to (51.4, 30.8)
- moved TP7 0.22 mm to (59.0, 32.0)
- moved R29 0.10 mm to (36.1, 26.1)
- moved S1 0.05 mm to (28.7, 24.0)
Routing:
- net +3V3: track 42.1 -> 38.9 mm, vias 37 -> 38
- net GND: track 57.7 -> 59.8 mm, vias 221 -> 219
- net /LCD_TE: track 16.1 -> 15.0 mm, vias 3 -> 2
Other:
- board text added: "JLCJLCJLCJLC"

Commit message: Initial PCB V1.1 changes
Parts:
- J3: value UART -> UART0
- L6: footprint Resistor_SMD:R_0402_1005Metric -> Inductor_SMD:L_0402_1005Metric
- Q1: value DMC2053UVT -> DMC2710UDW
- TP7: value UBX_RST -> GNSS Reset
Other:
- board text added: "ESPWatchS3 V1.1 Design By: Sam Bach"
- board text removed: "ESPWatchS3 V1.0 Design By: Sam Bach"
Changed lines of the file:
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@@
       (pintype "passive+no_connect"))
     (model "${KIPRJMOD}/Libraries/3D/EVQ-P4HB3B.step"
-      (offset (xyz 0 -1.9 1.6))
+      (offset (xyz 0 -1.6 -0.4))
       (scale (xyz 1 1 1))
-      (rotate (xyz -90 0 0))
+      (rotate (xyz 90 0 -180))
     )
   )
@@
         (effects (font (size 1 1) (thickness 0.15)))
     )
-    (fp_text value "UART" (at 0.17 -2.535 90) (layer "F.SilkS")
+    (fp_text value "UART0" (at 0.17 -2.535 90) (layer "F.SilkS")
         (effects (font (size 0.8 0.8) (thickness 0.1)))
     )
@@
     (property "ki_description" "test point")
     (property "ki_keywords" "test point tp")
-    (attr exclude_from_pos_files exclude_from_bom)
+    (attr exclude_from_pos_files)
     (fp_text reference "TP7" (at 0 -1.448) (layer "F.SilkS") hide
         (effects (font (size 1 1) (thickness 0.15)))
     )
-    (fp_text value "UBX_RST" (at 1.45 1.1 90) (layer "F.SilkS")
+    (fp_text value "GNSS Reset" (at 1.45 1.1 90) (layer "F.SilkS")
         (effects (font (size 0.8 0.8) (thickness 0.1)))
     )
@@
     (property "ki_description" "test point")
     (property "ki_keywords" "test point tp")
-    (attr exclude_from_pos_files exclude_from_bom)
+    (attr exclude_from_pos_files)
     (fp_text reference "TP8" (at 0 -1.448) (layer "F.SilkS") hide
         (effects (font (size 1 1) (thickness 0.15)))
@@
       (pintype "passive+no_connect"))
     (model "${KIPRJMOD}/Libraries/3D/EVQ-P4HB3B.step"
-      (offset (xyz 0 -1.9 1.6))
+      (offset (xyz 0 -1.6 -0.4))
       (scale (xyz 1 1 1))
-      (rotate (xyz -90 0 0))
+      (rotate (xyz 90 0 -180))
     )
   )
@@
     (property "ki_description" "test point")
     (property "ki_keywords" "test point tp")
-    (attr exclude_from_pos_files exclude_from_bom)
+    (attr exclude_from_pos_files)
     (fp_text reference "TP4" (at 0 -1.448) (layer "F.SilkS") hide
         (effects (font (size 1 1) (thickness 0.15)))
@@
     (property "ki_description" "test point")
     (property "ki_keywords" "test point tp")
-    (attr exclude_from_pos_files exclude_from_bom)
+    (attr exclude_from_pos_files)
     (fp_text reference "TP5" (at 0 -1.448) (layer "F.SilkS") hide
         (effects (font (size 1 1) (thickness 0.15)))
@@
       (pintype "passive+no_connect"))
     (model "${KIPRJMOD}/Libraries/3D/EVQ-P4HB3B.step"
-      (offset (xyz 0 -1.9 1.6))
+      (offset (xyz 0 -1.6 -0.4))
       (scale (xyz 1 1 1))
-      (rotate (xyz -90 0 0))
+      (rotate (xyz 90 0 -180))
     )
   )
@@
     (property "ki_description" "test point")
     (property "ki_keywords" "test point tp")
-    (attr exclude_from_pos_files exclude_from_bom)
+    (attr exclude_from_pos_files)
     (fp_text reference "TP3" (at 0 -1.448) (layer "F.SilkS") hide
         (effects (font (size 1 1) (thickness 0.15)))
@@
     (property "ki_description" "test point")
     (property "ki_keywords" "test point tp")
-    (attr exclude_from_pos_files exclude_from_bom)
+    (attr exclude_from_pos_files)
     (fp_text reference "TP2" (at 0 -1.448) (layer "F.SilkS") hide
         (effects (font (size 1 1) (thickness 0.15)))
@@
     )
   )
-  (footprint "Resistor_SMD:R_0402_1005Metric" (layer "F.Cu")
+  (footprint "Inductor_SMD:L_0402_1005Metric" (layer "F.Cu")
     (at 51.9 20.69 90)
-    (descr "Resistor SMD 0402 (1005 Metric), square (rectangular) end terminal, IPC_7351 nominal, (Body size source: IPC-SM-782 page 72, https://www.pcb-3d.com/wordpress/wp-content/uploads/ipc-sm-782a_amendment_1_and_2.pdf), generated with kicad-footprint-generator")
-    (tags "resistor")
+    (descr "Inductor SMD 0402 (1005 Metric), square (rectangular) end terminal, IPC_7351 nominal, (Body size source: http://www.tortai-tech.com/upload/download/2011102023233369053.pdf), generated with kicad-footprint-generator")
+    (tags "inductor")
     (property "Sheetfile" "ESPWatchS3.kicad_sch")
     (property "Sheetname" "")
@@
     (property "ki_keywords" "inductor choke coil reactor magnetic")
     (attr smd)
-    (fp_text reference "L6" (at 0 -1.17 90) (layer "F.SilkS") hide
+    (fp_text reference "L6" (at 0 -1.17 90) (layer "F.SilkS")
         (effects (font (size 1 1) (thickness 0.15)))
     )
@@
     )
     (fp_text user "${REFERENCE}" (at 0 0 90) (layer "F.Fab")
-        (effects (font (size 0.26 0.26) (thickness 0.04)))
+        (effects (font (size 0.25 0.25) (thickness 0.04)))
     )
-    (fp_line (start -0.153641 -0.38) (end 0.153641 -0.38)
-      (stroke (width 0.12) (type solid)) (layer "F.SilkS"))
-    (fp_line (start -0.153641 0.38) (end 0.153641 0.38)
-      (stroke (width 0.12) (type solid)) (layer "F.SilkS"))
     (fp_line (start -0.93 -0.47) (end 0.93 -0.47)
       (stroke (width 0.05) (type solid)) (layer "F.CrtYd"))
@@
     (fp_line (start 0.93 0.47) (end -0.93 0.47)
       (stroke (width 0.05) (type solid)) (layer "F.CrtYd"))
-    (fp_line (start -0.525 -0.27) (end 0.525 -0.27)
+    (fp_line (start -0.5 -0.25) (end 0.5 -0.25)
       (stroke (width 0.1) (type solid)) (layer "F.Fab"))
-    (fp_line (start -0.525 0.27) (end -0.525 -0.27)
+    (fp_line (start -0.5 0.25) (end -0.5 -0.25)
       (stroke (width 0.1) (type solid)) (layer "F.Fab"))
-    (fp_line (start 0.525 -0.27) (end 0.525 0.27)
+    (fp_line (start 0.5 -0.25) (end 0.5 0.25)
       (stroke (width 0.1) (type solid)) (layer "F.Fab"))
-    (fp_line (start 0.525 0.27) (end -0.525 0.27)
+    (fp_line (start 0.5 0.25) (end -0.5 0.25)
       (stroke (width 0.1) (type solid)) (layer "F.Fab"))
-    (pad "1" smd roundrect (at -0.51 0 90) (size 0.54 0.64) (layers "F.Cu" "F.Paste" "F.Mask") (roundrect_rratio 0.25)
+    (pad "1" smd roundrect (at -0.485 0 90) (size 0.59 0.64) (layers "F.Cu" "F.Paste" "F.Mask") (roundrect_rratio 0.25)
       (net 23 "Net-(U3-RF_IN)") (pintype "passive"))
-    (pad "2" smd roundrect (at 0.51 0 90) (size 0.54 0.64) (layers "F.Cu" "F.Paste" "F.Mask") (roundrect_rratio 0.25)
+    (pad "2" smd roundrect (at 0.485 0 90) (size 0.59 0.64) (layers "F.Cu" "F.Paste" "F.Mask") (roundrect_rratio 0.25)
       (net 124 "Net-(ANT2-PadFEED)") (pintype "passive"))
-    (model "${KICAD6_3DMODEL_DIR}/Resistor_SMD.3dshapes/R_0402_1005Metric.wrl"
+    (model "${KICAD6_3DMODEL_DIR}/Inductor_SMD.3dshapes/L_0402_1005Metric.wrl"
       (offset (xyz 0 0 0))
       (scale (xyz 1 1 1))
@@
       (pintype "passive+no_connect"))
     (model "${KIPRJMOD}/Libraries/3D/EVQ-P4HB3B.step"
-      (offset (xyz 0 -1.9 1.6))
+      (offset (xyz 0 -1.6 -0.4))
       (scale (xyz 1 1 1))
-      (rotate (xyz -90 0 0))
+      (rotate (xyz 90 0 -180))
     )
   )
@@
     (property "ki_description" "test point")
     (property "ki_keywords" "test point tp")
-    (attr exclude_from_pos_files exclude_from_bom)
+    (attr exclude_from_pos_files)
     (fp_text reference "TP6" (at 0 -1.448) (layer "F.SilkS") hide
         (effects (font (size 1 1) (thickness 0.15)))
@@
     (property "ki_description" "test point")
     (property "ki_keywords" "test point tp")
-    (attr exclude_from_pos_files exclude_from_bom)
+    (attr exclude_from_pos_files)
     (fp_text reference "TP1" (at 0 -1.448) (layer "F.SilkS") hide
         (effects (font (size 1 1) (thickness 0.15)))
@@
     (property "Sheetfile" "ESPWatchS3.kicad_sch")
     (property "Sheetname" "")
-    (property "ki_description" ".65A/-.6A Id, 20V Vds, Complementary pair enhancement mode P-Channel and N-Channel MOSFET, SOT-363-6")
+    (property "ki_description" ".65A/-.5A Id, 20V Vds, Complementary pair enhancement mode P-Channel and N-Channel MOSFET, SOT-363-6")
     (property "ki_keywords" "complementary mosfet")
     (attr smd)
@@
         (effects (font (size 1 1) (thickness 0.15)) (justify mirror))
     )
-    (fp_text value "DMC2053UVT" (at 0 -2) (layer "B.Fab") hide
+    (fp_text value "DMC2710UDW" (at 0 -2) (layer "B.Fab") hide
         (effects (font (size 1 1) (thickness 0.15)) (justify mirror))
     )
@@
   (gr_rect (start 43.205 40.59) (end 44.825 41.71)
     (stroke (width 0) (type solid)) (fill solid) (layer "F.Mask"))
-  (gr_line (start 44 57.5) (end 44 17.5)
-    (stroke (width 0.15) (type default)) (layer "Dwgs.User"))
-  (gr_line (start 27 37.5) (end 61 37.5)
-    (stroke (width 0.15) (type default)) (layer "Dwgs.User"))
   (gr_rect (start 27 17.5) (end 61 57.5)
     (stroke (width 0.1) (type default)) (fill none) (layer "Edge.Cuts"))
@@
     (effects (font (size 0.8 0.8) (thickness 0.1)) (justify left bottom))
   )
-  (gr_text "ESPWatchS3 \nV1.0\nDesign By:\nSam Bach" (at 32.45 50.5) (layer "F.SilkS")
+  (gr_text "ESPWatchS3 \nV1.1\nDesign By:\nSam Bach" (at 32.45 50.5) (layer "F.SilkS")
     (effects (font (size 0.8 0.8) (thickness 0.1)) (justify left bottom))
   )
@@
   (segment (start 34.85 40.45) (end 34.3 39.9) (width 0.3) (layer "B.Cu") (net 9))
   (segment (start 34.3 39.9) (end 33.15 39.9) (width 0.3) (layer "B.Cu") (net 9))
-  (segment (start 35.75 47.3) (end 34.85 46.4) (width 0.3) (layer "B.Cu") (net 9))
+  (segment (start 35.75 47.3) (end 34.85 46.4) (width 0.4) (layer "B.Cu") (net 9))
   (segment (start 33.15 39.9) (end 33.15 35.1) (width 0.5) (layer "B.Cu") (net 9))
   (segment (start 58.35 36) (end 58.95 35.4) (width 0.2) (layer "F.Cu") (net 10))
